File: test/test.sch (KiCad schematic (older format))
At the start: 16 parts, among them SW1 SW_SPST, U1 LM358P

Commit message: Trying out 5.0
Parts:
- BT1: symbol Battery -> Device:Battery
- BZ1: symbol PS1240P02BT -> test-rescue:PS1240P02BT
- C1: symbol C -> Device:C
- LED1: symbol LED -> Device:LED
- R1, R2, R3, R4, R5, R6, R7, R8, R9, RD1: symbol R -> Device:R
- SW1: symbol SW_SPST -> switches:SW_SPST
- U1: symbol LM358P -> test-rescue:LM358P
Changed lines of the file:
@@
-EESchema Schematic File Version 2
-LIBS:power
-LIBS:device
-LIBS:switches
-LIBS:relays
-LIBS:motors
-LIBS:transistors
-LIBS:conn
-LIBS:linear
-LIBS:regul
-LIBS:74xx
-LIBS:cmos4000
-LIBS:adc-dac
-LIBS:memory
-LIBS:xilinx
-LIBS:microcontrollers
-LIBS:dsp
-LIBS:microchip
-LIBS:analog_switches
-LIBS:motorola
-LIBS:texas
-LIBS:intel
-LIBS:audio
-LIBS:interface
-LIBS:digital-audio
-LIBS:philips
-LIBS:display
-LIBS:cypress
-LIBS:siliconi
-LIBS:opto
-LIBS:atmel
-LIBS:contrib
-LIBS:valves
-LIBS:oled
+EESchema Schematic File Version 4
 LIBS:test-cache
-EELAYER 25 0
+EELAYER 26 0
 EELAYER END
 $Descr A4 11693 8268
@@
 $EndDescr
 $Comp
-L GND #PWR01
+L power:GND #PWR01
 U 1 1 5AD74190
 P 3450 4500
@@
 $EndComp
 Wire Wire Line
-	3450 4500 6850 4500
+	3450 4500 4000 4500
 Wire Wire Line
 	6850 4500 8900 4550
@@
 Connection ~ 5650 4500
 $Comp
-L SW_SPST SW1
+L switches:SW_SPST SW1
 U 1 1 5AD74382
 P 6800 2850
@@
 $EndComp
 $Comp
-L LED LED1
+L Device:LED LED1
 U 1 1 5AD744BB
 P 4000 3300
@@
 $EndComp
 $Comp
-L R R1
+L Device:R R1
 U 1 1 5AD744F4
 P 4000 3000
@@
 $EndComp
 $Comp
-L R R3
+L Device:R R3
 U 1 1 5AD74539
 P 4500 3000
@@
 $EndComp
 Wire Wire Line
-	4000 2850 5650 2850
+	4000 2850 4500 2850
 Wire Wire Line
 	5650 2850 6300 3200
 $Comp
-L R R4
+L Device:R R4
 U 1 1 5AD892E5
 P 4500 4350
@@
 $EndComp
 $Comp
-L R R2
+L Device:R R2
 U 1 1 5AD8934C
 P 4000 4350
@@
 $EndComp
 $Comp
-L R R7
+L Device:R R7
 U 1 1 5AD893BF
 P 6600 3050
@@
 $EndComp
 $Comp
-L R R9
+L Device:R R9
 U 1 1 5AD89424
 P 7550 3500
@@
 $EndComp
 $Comp
-L R R6
+L Device:R R6
 U 1 1 5AD8946B
 P 6450 4350
@@
 $EndComp
 $Comp
-L R R5
+L Device:R R5
 U 1 1 5AD894E0
 P 6200 3650
@@
 $EndComp
 $Comp
-L R R8
+L Device:R R8
 U 1 1 5AD8985A
 P 6050 4000
@@
 $EndComp
 $Comp
-L PS1240P02BT BZ1
+L test-rescue:PS1240P02BT BZ1
 U 1 1 5AE1D2D9
 P 7650 4150
@@
 $EndComp
 Wire Wire Line
-	4000 3450 4000 4200
-Wire Wire Line
-	4500 3150 4500 4200
-Wire Wire Line
-	6450 3050 6450 4200
+	4000 3450 4000 3550
+Wire Wire Line
+	4500 3150 4500 3650
+Wire Wire Line
+	6450 3050 6450 3650
 Wire Wire Line
 	6350 3650 6450 3650
@@
 	6750 3050 6850 3050
 Wire Wire Line
-	6850 3050 6850 3550
+	6850 3050 6850 3450
 Connection ~ 6850 3450
 Wire Wire Line
@@
 Connection ~ 4500 3650
 $Comp
-L C C1
+L Device:C C1
 U 1 1 5AE1D652
 P 5350 4350
@@
 $EndComp
 Wire Wire Line
-	5150 4200 6350 4200
+	5150 4200 5350 4200
 Wire Wire Line
 	5150 4200 5150 3750
@@
 Connection ~ 6450 4500
 Connection ~ 6450 3650
-Connection ~ 5650 4150
 Connection ~ 6050 3850
 Text Notes 4900 2450 0    60   ~ 0
@@
 	6850 3850 7450 4050
 $Comp
-L GND #PWR02
+L power:GND #PWR02
 U 1 1 5B19D001
 P 8900 4550
@@
 $EndComp
 $Comp
-L LM358P U1
+L test-rescue:LM358P U1
 U 1 1 5AD740CD
 P 5750 3650
@@
 $EndComp
 $Comp
-L PWR_FLAG #FLG03
+L power:PWR_FLAG #FLG03
 U 1 1 5B19D68B
 P 7350 2850
@@
 $EndComp
 $Comp
-L +9V #PWR04
+L power:+9V #PWR04
 U 1 1 5B19D845
 P 7850 2850
@@
 Connection ~ 7350 2850
 Wire Wire Line
-	7000 2850 8300 2850
+	7000 2850 7350 2850
 Wire Wire Line
 	6300 3200 6300 2850
@@
 	6850 3850 7550 3650
 $Comp
-L PWR_FLAG #FLG05
+L power:PWR_FLAG #FLG05
 U 1 1 5B1A0048
 P 8900 4550
@@
 $EndComp
 $Comp
-L Battery BT1
+L Device:Battery BT1
 U 1 1 5B1A0D05
 P 8300 3400
@@
 Wire Wire Line
 	8300 4350 8900 4550
-Connection ~ 6300 2850
-Connection ~ 7000 2850
-$Comp
-L R RD1
+$Comp
+L Device:R RD1
 U 1 1 5B91D060
 P 6450 2850
@@
 Wire Wire Line
 	6100 3850 6050 3850
+Wire Wire Line
+	5650 4500 6450 4500
+Wire Wire Line
+	6450 4100 6450 4200
+Wire Wire Line
+	6850 3450 6850 3550
+Wire Wire Line
+	4000 3550 4000 4200
+Wire Wire Line
+	4500 3650 4500 4200
+Wire Wire Line
+	4500 2850 5650 2850
+Wire Wire Line
+	5350 4500 5650 4500
+Wire Wire Line
+	5350 4200 6350 4200
+Wire Wire Line
+	4500 4500 5350 4500
+Wire Wire Line
+	4000 4500 4500 4500
+Wire Wire Line
+	6450 4500 6850 4500
+Wire Wire Line
+	6450 3650 6450 4100
+Wire Wire Line
+	7350 2850 7850 2850
+Wire Wire Line
+	7850 2850 8300 2850
 $EndSCHEMATC

Commit message: Updated 7/2/20119 during meeting at RRFC
Parts:
- added H1, H2, H3, H4: MountingHole, MountingHole:MountingHole_2.2mm_M2, symbol Mechanical:MountingHole
- BZ1: symbol test-rescue:PS1240P02BT -> test-rescue:PS1240P02BT-test-rescue
- SW1: symbol switches:SW_SPST -> test-rescue:SW_SPST-switches
- U1: symbol test-rescue:LM358P -> test-rescue:LM358P-test-rescue
Changed lines of the file:
@@
 Connection ~ 5650 4500
 $Comp
-L switches:SW_SPST SW1
+L test-rescue:SW_SPST-switches SW1
 U 1 1 5AD74382
 P 6800 2850
@@
 $EndComp
 $Comp
-L test-rescue:PS1240P02BT BZ1
+L test-rescue:PS1240P02BT-test-rescue BZ1
 U 1 1 5AE1D2D9
 P 7650 4150
@@
 $EndComp
 $Comp
-L test-rescue:LM358P U1
+L test-rescue:LM358P-test-rescue U1
 U 1 1 5AD740CD
 P 5750 3650
@@
 Wire Wire Line
 	7850 2850 8300 2850
+$Comp
+L Mechanical:MountingHole H1
+U 1 1 5C5C9B1B
+P 3150 2550
+F 0 "H1" H 3250 2596 50  0000 L CNN
+F 1 "MountingHole" H 3250 2505 50  0000 L CNN
+F 2 "MountingHole:MountingHole_2.2mm_M2" H 3150 2550 50  0001 C CNN
+F 3 "~" H 3150 2550 50  0001 C CNN
+	1    3150 2550
+	1    0    0    -1
+$EndComp
+$Comp
+L Mechanical:MountingHole H2
+U 1 1 5C5C9BDD
+P 3200 4350
+F 0 "H2" H 3300 4396 50  0000 L CNN
+F 1 "MountingHole" H 3300 4305 50  0000 L CNN
+F 2 "MountingHole:MountingHole_2.2mm_M2" H 3200 4350 50  0001 C CNN
+F 3 "~" H 3200 4350 50  0001 C CNN
+	1    3200 4350
+	1    0    0    -1
+$EndComp
+$Comp
+L Mechanical:MountingHole H3
+U 1 1 5C5C9C45
+P 8950 2500
+F 0 "H3" H 9050 2546 50  0000 L CNN
+F 1 "MountingHole" H 9050 2455 50  0000 L CNN
+F 2 "MountingHole:MountingHole_2.2mm_M2" H 8950 2500 50  0001 C CNN
+F 3 "~" H 8950 2500 50  0001 C CNN
+	1    8950 2500
+	1    0    0    -1
+$EndComp
+$Comp
+L Mechanical:MountingHole H4
+U 1 1 5C5C9CBF
+P 9250 4350
+F 0 "H4" H 9350 4396 50  0000 L CNN
+F 1 "MountingHole" H 9350 4305 50  0000 L CNN
+F 2 "MountingHole:MountingHole_2.2mm_M2" H 9250 4350 50  0001 C CNN
+F 3 "~" H 9250 4350 50  0001 C CNN
+	1    9250 4350
+	1    0    0    -1
+$EndComp
 $EndSCHEMATC
